Commit message: Modified controller groups

File: fairino_description/urdf/fairino5_v6.urdf (robot description, URDF)
Before this commit: robot fairino5_v6_robot, 9 links, 8 joints
Joints:
- joint Ext_Axis: origin xyz=0 0 0 rpy=0 0 0 -> xyz=0 0 0.065 rpy=0 0 0

Commit message: Add gripper to robot description

File: fairino_description/urdf/fairino5_v6.urdf (robot description, URDF)
Before this commit: robot fairino5_v6_robot, 7 links, 6 joints
Links:
- added link hand; collision mesh filename=package://fairino_description/meshes/fairino5_v6/hand.dae; visual mesh filename=package://fairino_description/meshes/fairino5_v6/hand.dae
- added link leftfinger; collision mesh filename=package://fairino_description/meshes/fairino5_v6/finger.dae; visual mesh filename=package://fairino_description/meshes/fairino5_v6/finger.dae
- added link rightfinger; collision mesh filename=package://fairino_description/meshes/fairino5_v6/finger.dae; visual mesh filename=package://fairino_description/meshes/fairino5_v6/finger.dae
Joints:
- added joint finger_joint1: type prismatic, parent hand, child leftfinger, origin xyz=0 0 0.0584 rpy=0 0 0, axis 0 1 0, limit lower=0.0 upper=0.04 effort=20 velocity=0.2
- added joint finger_joint2: type prismatic, parent hand, child rightfinger, origin xyz=0 0 0.0584 rpy=0 0 0, axis 0 -1 0, limit lower=0.0 upper=0.04 effort=20 velocity=0.2, mimic joint=finger_joint1
- added joint gripper_joint: type fixed, parent wrist3_link, child hand, origin xyz=0 0 0.1 rpy=0 0 -0.785398163397

File: fr5_arm_hand_config/config/fairino5_v6_robot.urdf.xacro (robot description, xacro)
@@ -2,11 +2,8 @@
 <robot xmlns:xacro="http://www.ros.org/wiki/xacro" name="fairino5_v6_robot">
     <xacro:arg name="initial_positions_file" default="initial_positions.yaml" />
-    <xacro:arg name="ros2_control_hardware_type" default="mock_components" />
     <!-- Import fairino5_v6_robot urdf file -->
     <xacro:include filename="$(find fairino_description)/urdf/fairino5_v6.urdf" />
     <!-- Import control_xacro -->
     <xacro:include filename="fairino5_v6_robot.ros2_control.xacro" />
-    <xacro:include filename="hand.ros2_control.xacro" />
     <xacro:fairino5_v6_robot_ros2_control name="FakeSystem" initial_positions_file="$(arg initial_positions_file)"/>
-    <xacro:hand_ros2_control name="HandFakeSystem" ros2_control_hardware_type="$(arg ros2_control_hardware_type)"/>
 </robot>
