Commit message: First commit

File: fairino5_v6_moveit2_config/config/fairino5_v6_robot.ros2_control.xacro (robot description, xacro)
@@ -7,5 +7,4 @@
                 <!-- By default, set up controllers for simulation. This won't work on real hardware -->
                 <plugin>mock_components/GenericSystem</plugin>
-                <!-- <plugin>fairino_hardware/FairinoHardwareInterface</plugin> -->
             </hardware>
             <joint name="j1">
@@ -45,4 +44,10 @@
                 </state_interface>
             </joint>
+            <joint name="Ext_Axis">
+                <command_interface name="position"/>
+                <state_interface name="position">
+                  <param name="initial_value">${initial_positions['Ext_Axis']}</param>
+                </state_interface>
+            </joint>
         </ros2_control>
     </xacro:macro>

File: fairino_description/urdf/fairino5_v6.urdf (robot description, URDF)
Before this commit: robot fairino5_v6_robot, 7 links, 6 joints
Links:
- added link ext_axis_link, mass 10.0; collision box size=5.0 0.1 0.1; visual box size=5.0 0.1 0.1
- added link world
Joints:
- added joint Ext_Axis: type prismatic, parent ext_axis_link, child base_link, origin xyz=0 0 0 rpy=0 0 0, axis 1 0 0, limit lower=0.0 upper=5.0 effort=1000.0 velocity=1.0
- added joint world_to_ext_axis: type fixed, parent world, child ext_axis_link, origin xyz=0 0 0 rpy=0 0 0

Commit message: feat: integrate gripper control into hardware interface with moveit

File: fairino5_v6_moveit2_config/config/fairino5_v6_robot.ros2_control.xacro (robot description, xacro)
@@ -1,11 +1,14 @@
 <?xml version="1.0"?>
 <robot xmlns:xacro="http://www.ros.org/wiki/xacro">
-    <xacro:macro name="fairino5_v6_robot_ros2_control" params="name initial_positions_file">
-        <xacro:property name="initial_positions" value="${load_yaml(initial_positions_file)['initial_positions']}"/>
+    <xacro:macro name="fairino5_v6_robot_ros2_control" params="name initial_positions_file ros2_control_hardware_type">
+        <xacro:property name="initial_positions" value="${xacro.load_yaml(initial_positions_file)['initial_positions']}"/>
         <ros2_control name="${name}" type="system">
             <hardware>
-                <!-- By default, set up controllers for simulation. This won't work on real hardware -->
-                <plugin>mock_components/GenericSystem</plugin>
-                <!-- <plugin>fairino_hardware/FairinoHardwareInterface</plugin> -->
+                <xacro:if value="${ros2_control_hardware_type == 'mock_components'}">
+                    <plugin>mock_components/GenericSystem</plugin>
+                </xacro:if>
+                <xacro:if value="${ros2_control_hardware_type == 'Fr5Hardware'}">
+                    <plugin>fairino_hardware/FairinoHardwareInterface</plugin>
+                </xacro:if>
             </hardware>
             <joint name="j1">

File: fairino5_v6_moveit2_config/config/fairino5_v6_robot.urdf.xacro (robot description, xacro)
@@ -2,5 +2,8 @@
 <robot xmlns:xacro="http://www.ros.org/wiki/xacro" name="fairino5_v6_robot">
     <xacro:arg name="initial_positions_file" default="initial_positions.yaml" />
-    <xacro:arg name="ros2_control_hardware_type" default="mock_components" />
+    <!--Enable to use mock HW-->
+    <!-- <xacro:arg name="ros2_control_hardware_type" default="mock_components" /> -->
+    <!--Enable to use real HW-->
+    <xacro:arg name="ros2_control_hardware_type" default="Fr5Hardware" />
     <!-- Import fairino5_v6_robot urdf file -->
     <xacro:include filename="$(find fairino_description)/urdf/fairino5_v6.urdf" />
@@ -8,5 +11,8 @@
     <xacro:include filename="fairino5_v6_robot.ros2_control.xacro" />
     <xacro:include filename="hand.ros2_control.xacro" />
-    <xacro:fairino5_v6_robot_ros2_control name="FakeSystem" initial_positions_file="$(arg initial_positions_file)"/>
-    <xacro:hand_ros2_control name="HandFakeSystem" ros2_control_hardware_type="$(arg ros2_control_hardware_type)"/>
+    <!-- <xacro:fairino5_v6_robot_ros2_control name="FakeSystem" initial_positions_file="$(arg initial_positions_file)"/> -->
+    <xacro:fairino5_v6_robot_ros2_control name="Fr5Hardware" initial_positions_file="$(arg initial_positions_file)"
+                                                     ros2_control_hardware_type="$(arg ros2_control_hardware_type)"/>
+    <!-- <xacro:hand_ros2_control name="HandFakeSystem" ros2_control_hardware_type="$(arg ros2_control_hardware_type)"/> -->
+    <!-- <xacro:hand_ros2_control name="Fr5Hardware" ros2_control_hardware_type="$(arg ros2_control_hardware_type)"/>         -->
 </robot>

File: fr5_arm_hand_config/config/fairino5_v6_robot.ros2_control.xacro (robot description, xacro)
@@ -1,10 +1,14 @@
 <?xml version="1.0"?>
 <robot xmlns:xacro="http://www.ros.org/wiki/xacro">
-    <xacro:macro name="fairino5_v6_robot_ros2_control" params="name initial_positions_file">
-        <xacro:property name="initial_positions" value="${load_yaml(initial_positions_file)['initial_positions']}"/>
+    <xacro:macro name="fairino5_v6_robot_ros2_control" params="name initial_positions_file ros2_control_hardware_type">
+        <xacro:property name="initial_positions" value="${xacro.load_yaml(initial_positions_file)['initial_positions']}"/>
         <ros2_control name="${name}" type="system">
             <hardware>
-                <!-- By default, set up controllers for simulation. This won't work on real hardware -->
-                <plugin>mock_components/GenericSystem</plugin>
+                <xacro:if value="${ros2_control_hardware_type == 'mock_components'}">
+                    <plugin>mock_components/GenericSystem</plugin>
+                </xacro:if>
+                <xacro:if value="${ros2_control_hardware_type == 'Fr5Hardware'}">
+                    <plugin>fairino_hardware/FairinoHardwareInterface</plugin>
+                </xacro:if>
             </hardware>
             <joint name="j1">
@@ -13,5 +17,4 @@
                   <param name="initial_value">${initial_positions['j1']}</param>
                 </state_interface>
-                <state_interface name="velocity"/>
             </joint>
             <joint name="j2">
@@ -20,5 +23,4 @@
                   <param name="initial_value">${initial_positions['j2']}</param>
                 </state_interface>
-                <state_interface name="velocity"/>
             </joint>
             <joint name="j3">
@@ -27,5 +29,4 @@
                   <param name="initial_value">${initial_positions['j3']}</param>
                 </state_interface>
-                <state_interface name="velocity"/>
             </joint>
             <joint name="j4">
@@ -34,5 +35,4 @@
                   <param name="initial_value">${initial_positions['j4']}</param>
                 </state_interface>
-                <state_interface name="velocity"/>
             </joint>
             <joint name="j5">
@@ -41,5 +41,4 @@
                   <param name="initial_value">${initial_positions['j5']}</param>
                 </state_interface>
-                <state_interface name="velocity"/>
             </joint>
             <joint name="j6">
@@ -48,10 +47,20 @@
                   <param name="initial_value">${initial_positions['j6']}</param>
                 </state_interface>
-                <state_interface name="velocity"/>
             </joint>
+            <!-- Gripper joints - names MUST match URDF joint names exactly -->
             <joint name="finger_joint1">
                 <command_interface name="position"/>
                 <state_interface name="position">
                   <param name="initial_value">${initial_positions['finger_joint1']}</param>
+                </state_interface>
+                <!-- velocity required by GripperActionController (dummy value) -->
+                <state_interface name="velocity"/>
+            </joint>
+            <joint name="finger_joint2">
+                <param name="mimic">finger_joint1</param>
+                <param name="multiplier">1</param>
+                <command_interface name="position"/>
+                <state_interface name="position">
+                  <param name="initial_value">0.0</param>
                 </state_interface>
                 <state_interface name="velocity"/>

File: fr5_arm_hand_config/config/fairino5_v6_robot.urdf.xacro (robot description, xacro)
@@ -2,8 +2,14 @@
 <robot xmlns:xacro="http://www.ros.org/wiki/xacro" name="fairino5_v6_robot">
     <xacro:arg name="initial_positions_file" default="initial_positions.yaml" />
+    <!--Enable to use mock HW-->
+    <!-- <xacro:arg name="ros2_control_hardware_type" default="mock_components" /> -->
+    <!--Enable to use real HW-->
+    <xacro:arg name="ros2_control_hardware_type" default="Fr5Hardware" />
     <!-- Import fairino5_v6_robot urdf file -->
     <xacro:include filename="$(find fairino_description)/urdf/fairino5_v6.urdf" />
     <!-- Import control_xacro -->
     <xacro:include filename="fairino5_v6_robot.ros2_control.xacro" />
-    <xacro:fairino5_v6_robot_ros2_control name="FakeSystem" initial_positions_file="$(arg initial_positions_file)"/>
+    <!-- <xacro:fairino5_v6_robot_ros2_control name="FakeSystem" initial_positions_file="$(arg initial_positions_file)"/> -->
+    <xacro:fairino5_v6_robot_ros2_control name="Fr5Hardware" initial_positions_file="$(arg initial_positions_file)"
+                                                     ros2_control_hardware_type="$(arg ros2_control_hardware_type)"/>
 </robot>

Commit message: Add octomap configuration for 336L

File: fairino5_v6_moveit2_config/config/fairino5_v6_robot.ros2_control.xacro (robot description, xacro)
@@ -1,14 +1,10 @@
 <?xml version="1.0"?>
 <robot xmlns:xacro="http://www.ros.org/wiki/xacro">
-    <xacro:macro name="fairino5_v6_robot_ros2_control" params="name initial_positions_file ros2_control_hardware_type">
-        <xacro:property name="initial_positions" value="${xacro.load_yaml(initial_positions_file)['initial_positions']}"/>
+    <xacro:macro name="fairino5_v6_robot_ros2_control" params="name initial_positions_file">
+        <xacro:property name="initial_positions" value="${load_yaml(initial_positions_file)['initial_positions']}"/>
         <ros2_control name="${name}" type="system">
             <hardware>
-                <xacro:if value="${ros2_control_hardware_type == 'mock_components'}">
-                    <plugin>mock_components/GenericSystem</plugin>
-                </xacro:if>
-                <xacro:if value="${ros2_control_hardware_type == 'Fr5Hardware'}">
-                    <plugin>fairino_hardware/FairinoHardwareInterface</plugin>
-                </xacro:if>
+                <!-- By default, set up controllers for simulation. This won't work on real hardware -->
+                <plugin>mock_components/GenericSystem</plugin>
             </hardware>
             <joint name="j1">
@@ -48,4 +44,11 @@
                 </state_interface>
             </joint>
+            <joint name="finger_joint1">
+                <command_interface name="position"/>
+                <state_interface name="position">
+                  <param name="initial_value">${initial_positions['finger_joint1']}</param>
+                </state_interface>
+                <state_interface name="velocity"/>
+            </joint>
         </ros2_control>
     </xacro:macro>

File: fairino5_v6_moveit2_config/config/fairino5_v6_robot.urdf.xacro (robot description, xacro)
@@ -2,17 +2,9 @@
 <robot xmlns:xacro="http://www.ros.org/wiki/xacro" name="fairino5_v6_robot">
     <xacro:arg name="initial_positions_file" default="initial_positions.yaml" />
-    <!--Enable to use mock HW-->
-    <!-- <xacro:arg name="ros2_control_hardware_type" default="mock_components" /> -->
-    <!--Enable to use real HW-->
-    <xacro:arg name="ros2_control_hardware_type" default="Fr5Hardware" />
     <!-- Import fairino5_v6_robot urdf file -->
-    <xacro:include filename="$(find fairino_description)/urdf/fairino5_v6.urdf" />
+    <!-- <xacro:include filename="$(find fairino_description)/urdf/fairino5_v6.urdf" /> -->
+    <xacro:include filename="$(find fairino_description)/urdf/fairino5_v6_with_camera.urdf.xacro" />
     <!-- Import control_xacro -->
     <xacro:include filename="fairino5_v6_robot.ros2_control.xacro" />
-    <xacro:include filename="hand.ros2_control.xacro" />
-    <!-- <xacro:fairino5_v6_robot_ros2_control name="FakeSystem" initial_positions_file="$(arg initial_positions_file)"/> -->
-    <xacro:fairino5_v6_robot_ros2_control name="Fr5Hardware" initial_positions_file="$(arg initial_positions_file)"
-                                                     ros2_control_hardware_type="$(arg ros2_control_hardware_type)"/>
-    <!-- <xacro:hand_ros2_control name="HandFakeSystem" ros2_control_hardware_type="$(arg ros2_control_hardware_type)"/> -->
-    <!-- <xacro:hand_ros2_control name="Fr5Hardware" ros2_control_hardware_type="$(arg ros2_control_hardware_type)"/>         -->
+    <xacro:fairino5_v6_robot_ros2_control name="FakeSystem" initial_positions_file="$(arg initial_positions_file)"/>
 </robot>

File: fr5_arm_hand_config/config/fairino5_v6_robot.urdf.xacro (robot description, xacro)
@@ -7,5 +7,6 @@
     <xacro:arg name="ros2_control_hardware_type" default="Fr5Hardware" />
     <!-- Import fairino5_v6_robot urdf file -->
-    <xacro:include filename="$(find fairino_description)/urdf/fairino5_v6.urdf" />
+    <!-- <xacro:include filename="$(find fairino_description)/urdf/fairino5_v6.urdf" /> -->
+    <xacro:include filename="$(find fairino_description)/urdf/fairino5_v6_with_camera.urdf.xacro" />
     <!-- Import control_xacro -->
     <xacro:include filename="fairino5_v6_robot.ros2_control.xacro" />
