Commit message: feat: add camera mount URDF, fr5_motion_cpp package, MTC pick & place controller
- Add camera mount meshes (STL) and URDF xacro for Fairino5 with camera
- New fr5_motion_cpp package: MoveGroupInterface C++ node + headless launch
- Add MTC pick & place controller (pick_place_controller.cpp)
- Add sim.launch.py for MTC simulation testing
- Update fr5_arm_hand_config: SRDF, RViz, sensors, demo launch
- Update fairino5_v6_moveit2_config: ros2_control, URDF, kinematics, sensors
- Add FastDDS config (fastdds.xml, 4MB buffer)
- Update README and .claude config

Co-Authored-By: Claude Sonnet 4.6 <noreply@anthropic.com>

File: fairino5_v6_moveit2_config/config/fairino5_v6_robot.ros2_control.xacro (robot description, xacro)
@@ -7,4 +7,5 @@
                 <!-- By default, set up controllers for simulation. This won't work on real hardware -->
                 <plugin>mock_components/GenericSystem</plugin>
+                <!-- <plugin>fairino_hardware/FairinoHardwareInterface</plugin> -->
             </hardware>
             <joint name="j1">

File: fairino5_v6_moveit2_config/config/fairino5_v6_robot.urdf.xacro (robot description, xacro)
@@ -3,6 +3,6 @@
     <xacro:arg name="initial_positions_file" default="initial_positions.yaml" />
     <!-- Import fairino5_v6_robot urdf file -->
-    <!-- <xacro:include filename="$(find fairino_description)/urdf/fairino5_v6.urdf" /> -->
-    <xacro:include filename="$(find fairino_description)/urdf/fairino5_v6_with_camera.urdf.xacro" />
+    <xacro:include filename="$(find fairino_description)/urdf/fairino5_v6.urdf" />
+    <!-- <xacro:include filename="$(find fairino_description)/urdf/fairino5_v6_with_camera.urdf.xacro" /> -->
     <!-- Import control_xacro -->
     <xacro:include filename="fairino5_v6_robot.ros2_control.xacro" />

File: fairino_description/urdf/fairino5_v6_with_camera.urdf.xacro (robot description, xacro)
@@ -4,7 +4,9 @@
   <xacro:include filename="$(find fairino_description)/urdf/fairino5_v6_gripper.urdf.xacro" />
   <xacro:include filename="$(find fairino_description)/urdf/gemini335L_336L_camera.urdf.xacro" />
+  <xacro:include filename="$(find fairino_description)/urdf/camera_mount.urdf.xacro" />
   <link name="world" />
   <xacro:fairino5_v6_arm />
   <xacro:fairino5_v6_gripper />
+  <xacro:camera_mount />
   <xacro:gemini335L_336L_camera />
   <joint name="world_to_base_link" type="fixed">
@@ -13,13 +15,15 @@
     <origin xyz="0 0 0" rpy="0 0 0" />
   </joint>
-  <!-- <joint name="world_to_camera_link" type="fixed">
-    <parent link="world" />
+  <!-- Mount bracket attached to wrist3 -->
+  <joint name="wrist3_to_mount" type="fixed">
+    <parent link="wrist3_link" />
+    <child link="mount_base_link" />
+    <origin xyz="0 0 0.1" rpy="0 0 0.78539816339" />
+  </joint>
+  <!-- Camera attached to mount connector -->
+  <joint name="mount_to_camera" type="fixed">
+    <parent link="connector_link" />
     <child link="camera_link" />
-    <origin xyz="-0.3 -0.8 0.2" rpy="0 0 0.52359877559" />
-  </joint> -->
-  <joint name="camera_to_base" type="fixed">
-    <parent link="base_link"/>
-    <child link="camera_link"/>
-    <origin xyz="-0.5 -0.5 0.3" rpy="0 0 0.52359877559"/>  <!-- Tuỳ vị trí camera -->
+    <origin xyz="0 0 0.0235" rpy="0 -1.57079632679 1.57079632679" />
   </joint>
 </robot>
